File: PCB/atari_gravitar_bw_pcb/SheetMisc.kicad_sch (KiCad schematic)
At the start: 0 parts

Commit message: Sheet 3B complete
Parts:
- added J18: cat_connector, symbol atari:cat_connector
- added J19: J19_grav, symbol atari:J19_grav
- added J20: J20_grav, symbol atari:J20_grav
- added TPCAT_STROBE1: tp_2_pin, symbol atari:tp_2_pin
Connections:
- new net: J18.35 (CAT_STROBE), TPCAT_STROBE1.1, TPCAT_STROBE1.2
- new net +10V: J20.18 (+10_UNREG), J20.E (+10_UNREG)
- new net +24V: J20.3 (22VDC), J20.X (22VDC)
- new net +5V: J18.45 (5V0), J18.46 (5V0), J18.47 (5V0), J18.48 (5V0), J18.49 (5V0), J18.50 (5V0), J20.2 (+5V_REG), J20.21 (+SENSE), J20.B (+5V_REG), J20.Y (+5V_REG)
- new net -24V: J20.4 (-22VDC), J20.W (-22VDC)
- new net A0: J18.17 (A0)
- new net A1: J18.18 (A1)
- new net A10: J18.7 (A10)
- new net A11: J18.8 (A11)
- new net A12: J18.21 (A12)
- new net A13: J18.22 (A13)
- new net A14: J18.19 (A14)
- new net A15: J18.20 (A15)
- new net A2: J18.15 (A2)
- new net A3: J18.16 (A3)
- new net A4: J18.13 (A4)
- new net A5: J18.14 (A5)
- new net A6: J18.10 (A6), J18.11 (A6)
- new net A7: J18.12 (A7)
- new net A8: J18.9 (A8)
- new net AUD1: J19.12 (AUD1)
- new net AUD2: J19.11 (AUD2)
- new net BLUE: J19.9 (BLUE)
- new net CABINET: J20.R (CABINET)
- new net CNTR_L: J20.H (CNTR_L)
- new net CNTR_R: J20.6 (CNTR_R)
- new net COIN_AUX: J20.S (COIN_AUX)
- new net COIN_L: J20.16 (COIN_L)
- new net COIN_R: J20.U (COIN_R)
- new net D0: J18.29 (D0)
- new net D1: J18.30 (D1)
- new net D2: J18.27 (D2)
- new net D3: J18.28 (D3)
- new net D4: J18.25 (D4)
- new net D5: J18.26 (D5)
- new net D6: J18.23 (D6)
- new net D7: J18.24 (D7)
- new net FIRE1: J19.4 (FIRE1)
- new net FIRE2: J20.9 (FIRE2)
- new net GND: J18.1 (GND), J18.2 (GND), J18.3 (GND), J18.34 (PROMEN), J18.4 (GND), J18.5 (GND), J18.6 (GND), J19.1 (GND), J19.2 (GND), J19.H (GND), J19.J (GND), J19.K (GND), J19.L (GND), J19.M (GND), J20.1 (+5V_RTN), J20.12 (GND), J20.13 (GND), J20.22 (-SENSE), J20.A (+5V_RTN), J20.N (GND), J20.P (GND), J20.Z (+5V_RTN)
- new net GREEN: J19.8 (GREEN)
- new net LOCKOUT: J20.F (LOCKOUT)
- new net P1_LED: J20.7 (P1_LED)
- new net P2_LED: J20.J (P2_LED)
- new net PHI0: J18.33 (PHI0)
- new net PHI2: J18.31 (PHI2)
- new net RED: J19.7 (RED)
- new net ROT_LEFT1: J19.E (ROT_LEFT1)
- new net ROT_LEFT2: J20.8 (ROT_LEFT2)
- new net ROT_RIGHT1: J19.5 (ROT_RIGHT1)
- new net ROT_RIGHT2: J20.K (ROT_RIGHT2)
- new net R/~{W}: J18.32 (R/~{W})
- new net SELF_TEST: J20.T (SELF_TEST)
- new net SHIELDS1: J19.3 (SHIELDS1)
- new net SHIELDS2: J20.L (SHIELDS2)
- new net SLAM: J20.14 (SLAM)
- new net START1: J20.M (START1)
- new net START2: J20.11 (START2)
- new net THRUST1: J19.6 (THRUST1)
- new net THRUST2: J20.10 (THRUST2)
- new net X_OUT: J19.A (X_OUT)
- new net Y_OUT: J19.B (Y_OUT)
- new net Z_OUT: J19.10 (Z_OUT)
- new net ~{DISDAT}: J18.36 (~{DISDAT})
- new net ~{RESET}: J20.V (~{RESET})
- no-connect marks 0 -> 11

Commit message: Worked on the schematic library
Parts:
- J19: symbol atari:J19_grav -> atari:grav_J19
- J20: symbol atari:J20_grav -> atari:grav_J20
Changed lines of the file:
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@@
   (junction (at 166.37 64.135) (diameter 0) (color 0 0 0 0)
   )
-  (no_connect (at 140.97 41.275))
   (no_connect (at 140.97 43.815))
   (no_connect (at 140.97 64.135))
   (no_connect (at 140.97 48.895))
+  (no_connect (at 140.97 41.275))
   (no_connect (at 70.485 33.655))
   (no_connect (at 70.485 31.115))
@@
     (pin "1")
   )
-  (symbol (lib_id "atari:J19_grav") (at 120.65 50.165 0) (unit 1)
+  (symbol (lib_id "atari:grav_J19") (at 120.65 50.165 0) (unit 1)
     (in_bom yes) (on_board yes) (fields_autoplaced)
     (property "Reference" "J19" (id 0) (at 120.65 32.3555 0))
@@
     (pin "1")
   )
-  (symbol (lib_id "atari:J20_grav") (at 50.165 52.705 0) (unit 1)
+  (symbol (lib_id "atari:grav_J20") (at 50.165 52.705 0) (unit 1)
     (in_bom yes) (on_board yes) (fields_autoplaced)
     (property "Reference" "J20" (id 0) (at 50.165 22.1955 0))
