File: PCB/atari_gravitar_bw_pcb/atari_gravitar_bw_pcb.kicad_sch (KiCad schematic)
At the start: 0 parts

Commit message: Initial configuration
Changed lines of the file:
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@@
   )
   (text "Sheet3B" (at 16.51 38.1 0)
-    (effects (font (size 5.08 5.08) (thickness 0.254) bold) (justify left bottom))
+    (effects (font (size 5.08 5.08) (thickness 1.016) bold) (justify left bottom))
   )
   (text "Sheet7A" (at 61.595 127 0)
-    (effects (font (size 5.08 5.08) (thickness 0.254) bold) (justify left bottom))
+    (effects (font (size 5.08 5.08) (thickness 1.016) bold) (justify left bottom))
   )
   (text "Misc." (at 113.03 171.45 0)
-    (effects (font (size 5.08 5.08) (thickness 0.254) bold) (justify left bottom))
+    (effects (font (size 5.08 5.08) (thickness 1.016) bold) (justify left bottom))
   )
   (text "Sheet8B" (at 61.595 171.45 0)
-    (effects (font (size 5.08 5.08) (thickness 0.254) bold) (justify left bottom))
+    (effects (font (size 5.08 5.08) (thickness 1.016) bold) (justify left bottom))
   )
   (text "Sheet7B" (at 105.41 127 0)
-    (effects (font (size 5.08 5.08) (thickness 0.254) bold) (justify left bottom))
+    (effects (font (size 5.08 5.08) (thickness 1.016) bold) (justify left bottom))
   )
   (text "Sheet6A" (at 105.41 82.55 0)
-    (effects (font (size 5.08 5.08) (thickness 0.254) bold) (justify left bottom))
+    (effects (font (size 5.08 5.08) (thickness 1.016) bold) (justify left bottom))
   )
   (text "Sheet5B" (at 61.595 82.55 0)
-    (effects (font (size 5.08 5.08) (thickness 0.254) bold) (justify left bottom))
+    (effects (font (size 5.08 5.08) (thickness 1.016) bold) (justify left bottom))
   )
   (text "Sheet4B" (at 105.41 37.465 0)
-    (effects (font (size 5.08 5.08) (thickness 0.254) bold) (justify left bottom))
+    (effects (font (size 5.08 5.08) (thickness 1.016) bold) (justify left bottom))
   )
   (text "Sheet5A" (at 16.51 82.55 0)
-    (effects (font (size 5.08 5.08) (thickness 0.254) bold) (justify left bottom))
+    (effects (font (size 5.08 5.08) (thickness 1.016) bold) (justify left bottom))
   )
   (text "ARCADE PCB\nSCHEMATICS" (at 154.94 153.67 0)
@@
   )
   (text "Sheet4A" (at 61.595 38.1 0)
-    (effects (font (size 5.08 5.08) (thickness 0.254) bold) (justify left bottom))
+    (effects (font (size 5.08 5.08) (thickness 1.016) bold) (justify left bottom))
   )
   (text "Sheet8A" (at 16.51 171.45 0)
-    (effects (font (size 5.08 5.08) (thickness 0.254) bold) (justify left bottom))
+    (effects (font (size 5.08 5.08) (thickness 1.016) bold) (justify left bottom))
   )
   (text "Sheet6B" (at 16.51 127 0)
-    (effects (font (size 5.08 5.08) (thickness 0.254) bold) (justify left bottom))
+    (effects (font (size 5.08 5.08) (thickness 1.016) bold) (justify left bottom))
   )
   (sheet (at 103.505 104.775) (size 38.1 38.1) (fields_autoplaced)
