File: PCB/atari_gravitar_bw_pcb/Sheet4B.kicad_sch (KiCad schematic)
At the start: 0 parts

Commit message: Completed sheet 4b
Parts:
- added A_4: LM555, symbol atari:LM555
- added B_6: 74LS86, symbol atari:74LS86
- added C16: 47uf 50V, symbol Device:C_Polarized_US
- added C17, C36, C38: 10uf 50V, symbol Device:C_Polarized_US
- added C9: .1, symbol Device:C
- added CR1, CR2: 1N100, symbol Device:D
- added D_1, E/F_1, H_1, J_1, K/L_1, M_1: 2732, symbol atari:2732
- added E_2, H_2: 74LS244, symbol atari:74LS244
- added E_3: 74LS00, symbol atari:74LS00
- added J_2: 74LS374, symbol atari:74LS374
- added K_2: 74LS175, symbol atari:74LS175
- added L2, L3: 100uh, symbol Device:L
- added M_2: grav_nvram, symbol atari:grav_nvram
- added N/P_1: 6116, symbol atari:6116
- added P_2: 74LS174, symbol atari:74LS174
- added R1, R10, R11, R12, R13, R14, R15, R16, R17, R18, R2, R21, R3, R4, R5, R6, R7, R8, R9: 10k, symbol Device:R_US
- added TP-28V1: tp_2_pin, symbol atari:tp_2_pin
Connections:
- new net: M_2.11 (A1), P_2.7 (Q2), R1.1
- new net: C16.2, C9.1, CR1.2 (A), M_2.14 (VEE), TP-28V1.1, TP-28V1.2
- new net: K_2.2 (Q0), M_2.13 (CK), R11.1
- new net: H_2.13, J_2.6 (O2), M_2.20 (D0), R16.1
- new net: H_2.11, J_2.9 (O3), M_2.4 (D5), R15.1
- new net: H_2.15, J_2.5 (O1), M_2.21 (D1), R17.1
- new net: H_2.17, J_2.2 (O0), M_2.22 (D2), R18.1
- new net: H_2.2, J_2.19 (O7), M_2.2 (D7), R8.1
- new net: H_2.4, J_2.16 (O6), M_2.3 (D6), R7.1
- new net: H_2.6, J_2.15 (O5), M_2.5 (D4), R6.1
- new net: H_2.8, J_2.12 (O4), M_2.1 (D3), R9.1
- new net: M_2.12 (A0), P_2.10 (Q3), R10.1
- new net: D_1.10 (D1), E/F_1.10 (D1), E_2.17, H_1.10 (D1), J_1.10 (D1), K/L_1.10 (D1), M_1.10 (D1)
- new net: D_1.11 (D2), E/F_1.11 (D2), E_2.4, H_1.11 (D2), J_1.11 (D2), K/L_1.11 (D2), M_1.11 (D2)
- new net: D_1.13 (D3), E/F_1.13 (D3), E_2.15, H_1.13 (D3), J_1.13 (D3), K/L_1.13 (D3), M_1.13 (D3)
- new net: D_1.14 (D4), E/F_1.14 (D4), E_2.6, H_1.14 (D4), J_1.14 (D4), K/L_1.14 (D4), M_1.14 (D4)
- new net: D_1.15 (D5), E/F_1.15 (D5), E_2.13, H_1.15 (D5), J_1.15 (D5), K/L_1.15 (D5), M_1.15 (D5)
- new net: D_1.16 (D6), E/F_1.16 (D6), E_2.8, H_1.16 (D6), J_1.16 (D6), K/L_1.16 (D6), M_1.16 (D6)
- new net: D_1.17 (D7), E/F_1.17 (D7), E_2.11, H_1.17 (D7), J_1.17 (D7), K/L_1.17 (D7), M_1.17 (D7)
- new net: D_1.9 (D0), E/F_1.9 (D0), E_2.2, H_1.9 (D0), J_1.9 (D0), K/L_1.9 (D0), M_1.9 (D0)
- new net: A_4.3 (Q), C36.1
- new net: C36.2, CR1.1 (K), CR2.2 (A)
- new net: M_2.9 (A3), P_2.12 (Q4), R3.1
- new net: B_6.8, N/P_1.19 (A10)
- new net: A_4.8 (VCC), C17.1, L2.1
- new net: K_2.10 (Q2), M_2.16 (C2), R13.1
- new net: J_2.1 (OE), K_2.14 (~{Q3}), M_2.15 (C1), R12.1
- new net: K_2.7 (Q1), M_2.17 (CS1), R14.1
- new net: M_2.10 (A2), P_2.5 (Q1), R2.1
- new net: E_2.1 (1G), E_2.19 (2G), E_3.8
- new net: M_2.7 (A5), P_2.15 (Q5), R5.1
- new net: M_2.8 (A4), P_2.2 (Q0), R4.1
- new net: C16.1, C38.2, CR2.1 (K), L3.1
- new net +15V: L2.2
- new net +5V: D_1.21 (VPP), D_1.24 (VCC), E/F_1.21 (VPP), E/F_1.24 (VCC), E_2.20 (VCC), H_1.21 (VPP), H_1.24 (VCC), H_2.20 (VCC), J_1.21 (VPP), J_1.24 (VCC), J_2.20 (VCC), K/L_1.21 (VPP), K/L_1.24 (VCC), K_2.16 (VCC), M_1.21 (VPP), M_1.24 (VCC), M_2.6 (VSS), N/P_1.24 (VCC), P_2.16 (VCC), R1.2, R10.2, R11.2, R12.2, R13.2, R14.2, R15.2, R16.2, R17.2, R18.2, R2.2, R21.1, R3.2, R4.2, R5.2, R6.2, R7.2, R8.2, R9.2
- new net -15V: L3.2
- new net 12KHZ: A_4.4 (R)
- new net A10: B_6.9
- new net AB0: D_1.8 (A0), E/F_1.8 (A0), H_1.8 (A0), J_1.8 (A0), K/L_1.8 (A0), M_1.8 (A0), N/P_1.8 (A0), P_2.11 (D3)
- new net AB1: D_1.7 (A1), E/F_1.7 (A1), H_1.7 (A1), J_1.7 (A1), K/L_1.7 (A1), M_1.7 (A1), N/P_1.7 (A1), P_2.6 (D2)
- new net AB10: D_1.19 (A10), E/F_1.19 (A10), H_1.19 (A10), J_1.19 (A10), K/L_1.19 (A10), M_1.19 (A10)
- new net AB11: D_1.18 (A11), E/F_1.18 (A11), H_1.18 (A11), J_1.18 (A11), K/L_1.18 (A11), M_1.18 (A11)
- new net AB2: D_1.6 (A2), E/F_1.6 (A2), H_1.6 (A2), J_1.6 (A2), K/L_1.6 (A2), M_1.6 (A2), N/P_1.6 (A2), P_2.4 (D1)
- new net AB3: D_1.5 (A3), E/F_1.5 (A3), H_1.5 (A3), J_1.5 (A3), K/L_1.5 (A3), M_1.5 (A3), N/P_1.5 (A3), P_2.13 (D4)
- new net AB4: D_1.4 (A4), E/F_1.4 (A4), H_1.4 (A4), J_1.4 (A4), K/L_1.4 (A4), M_1.4 (A4), N/P_1.4 (A4), P_2.3 (D0)
- new net AB5: D_1.3 (A5), E/F_1.3 (A5), H_1.3 (A5), J_1.3 (A5), K/L_1.3 (A5), M_1.3 (A5), N/P_1.3 (A5), P_2.14 (D5)
- new net AB6: D_1.2 (A6), E/F_1.2 (A6), H_1.2 (A6), J_1.2 (A6), K/L_1.2 (A6), M_1.2 (A6), N/P_1.2 (A6)
- new net AB7: D_1.1 (A7), E/F_1.1 (A7), H_1.1 (A7), J_1.1 (A7), K/L_1.1 (A7), M_1.1 (A7), N/P_1.1 (A7)
- new net AB8: D_1.23 (A8), E/F_1.23 (A8), H_1.23 (A8), J_1.23 (A8), K/L_1.23 (A8), M_1.23 (A8), N/P_1.23 (A8)
- new net AB9: D_1.22 (A9), E/F_1.22 (A9), H_1.22 (A9), J_1.22 (A9), K/L_1.22 (A9), M_1.22 (A9), N/P_1.22 (A9)
- new net BANK_SEL: B_6.10
- new net D0: E_2.18
- new net D1: E_2.3
- new net D2: E_2.16
- new net D3: E_2.5
- new net D4: E_2.14
- new net D5: E_2.7
- new net D6: E_2.12
- new net D7: E_2.9
- new net DB0: H_2.7, J_2.7 (D2), K_2.4 (D0), N/P_1.9 (D0)
- new net DB1: H_2.5, J_2.4 (D1), K_2.12 (D2), N/P_1.10 (D1)
- new net DB2: H_2.3, J_2.3 (D0), K_2.13 (D3), N/P_1.11 (D2)
- new net DB3: H_2.12, J_2.13 (D4), K_2.5 (D1), N/P_1.13 (D3)
- new net DB4: H_2.14, J_2.14 (D5), N/P_1.14 (D4)
- new net DB5: H_2.9, J_2.8 (D3), N/P_1.15 (D5)
- new net DB6: H_2.16, J_2.17 (D6), N/P_1.16 (D6)
- new net DB7: H_2.18, J_2.18 (D7), N/P_1.17 (D7)
- new net GND: A_4.1 (GND), A_4.2 (TR), A_4.6 (THR), C17.2, C38.1, C9.2, D_1.12 (GND), E/F_1.12 (GND), E_2.10 (GND), H_1.12 (GND), H_2.10 (GND), J_1.12 (GND), J_2.10 (GND), K/L_1.12 (GND), K_2.8 (GND), M_1.12 (GND), M_2.18 (~{CS2}), M_2.19 (VSI), N/P_1.12 (GND), N/P_1.20 (~{OE}), P_2.8 (GND)
- new net PR23: P_2.1 (~{Mr})
- new net ROM: E_3.10
- new net ~{DISDAT}: E_3.9, R21.2
- new net ~{EAROMCON}: K_2.9 (Cp)
- new net ~{EAROMRD}: H_2.1 (1G), H_2.19 (2G)
- new net ~{EAROMWR}: J_2.11 (Cp), P_2.9 (Cp)
- new net ~{RAM}: N/P_1.18 (~{CE})
- new net ~{RESET}: K_2.1 (~{Mr})
- new net ~{ROM0}: D_1.20 (~{CS})
- new net ~{ROM1}: E/F_1.20 (~{CS})
- new net ~{ROM2}: H_1.20 (~{CS})
- new net ~{ROM3}: J_1.20 (~{CS})
- new net ~{ROM4}: K/L_1.20 (~{CS})
- new net ~{ROM5}: M_1.20 (~{CS})
- new net ~{WRITE}: N/P_1.21 (~{WE})
- no-connect marks 0 -> 6
Other:
- note added: "HIGH-SCORE TABLE"
- note added: "RANDOM-ACCESS MEMORY"
- note added: "READ-ONLY MEMORY"
