File: PCB/atari_gravitar_bw_pcb/Sheet6A.kicad_sch (KiCad schematic)
At the start: 0 parts

Commit message: Finished sheet 6A
Parts:
- added A_8, B_8, C_8, F_8, H_8, J_8: 74LS194, symbol atari:74LS194
- added C_6, D_6: 74LS175, symbol atari:74LS175
- added E_7: 74LS00, symbol atari:74LS00
- added F_7: 74LS14, symbol atari:74LS14
Connections:
- new net: A_8.10 (S1), C_8.10 (S1), E_7.11
- new net: A_8.9 (S0), C_8.9 (S0), F_7.10
- new net: B_8.10 (S1), E_7.8
- new net: B_8.9 (S0), F_7.8
- new net: F_7.2, H_8.9 (S0)
- new net: F_7.12, F_8.9 (S0), J_8.9 (S0)
- new net: E_7.3, F_8.10 (S1), J_8.10 (S1)
- new net: E_7.6, H_8.10 (S1)
- new net +5V: A_8.16 (VCC), B_8.16 (VCC), C_6.16 (VCC), C_8.16 (VCC), D_6.16 (VCC), E_7.14 (VCC), F_7.14 (VCC), F_8.16 (VCC), H_8.16 (VCC), J_8.16 (VCC)
- new net 12MHZ: A_8.11 (Cp), B_8.11 (Cp), C_8.11 (Cp), F_8.11 (Cp), H_8.11 (Cp), J_8.11 (Cp)
- new net DVG0: A_8.6 (P3), B_8.6 (P3), F_8.6 (P3), H_8.6 (P3)
- new net DVG1: A_8.5 (P2), B_8.5 (P2), F_8.5 (P2), H_8.5 (P2)
- new net DVG2: A_8.4 (P1), B_8.4 (P1), F_8.4 (P1), H_8.4 (P1)
- new net DVG3: A_8.3 (P0), B_8.3 (P0), F_8.3 (P0), H_8.3 (P0)
- new net DVG4: C_6.4 (D0), C_8.6 (P3), D_6.4 (D0), J_8.6 (P3)
- new net DVG5: C_6.5 (D1), C_8.5 (P2), D_6.5 (D1), J_8.5 (P2)
- new net DVG6: C_6.12 (D2), C_8.4 (P1), D_6.12 (D2), J_8.4 (P1)
- new net DVG7: C_6.13 (D3), C_8.3 (P0), D_6.13 (D3), J_8.3 (P0)
- new net DVX10: B_8.14 (Q1)
- new net DVX11: B_8.15 (Q0)
- new net DVX12: C_6.2 (Q0)
- new net DVX3: A_8.15 (Q0), C_8.7 (Dsl)
- new net DVX4: C_8.12 (Q3)
- new net DVX5: C_8.13 (Q2)
- new net DVX6: C_8.14 (Q1)
- new net DVX7: B_8.7 (Dsl), C_8.15 (Q0)
- new net DVX8: B_8.12 (Q3)
- new net DVX9: B_8.13 (Q2)
- new net DVY0: F_8.12 (Q3)
- new net DVY1: F_8.13 (Q2)
- new net DVY10: H_8.14 (Q1)
- new net DVY11: H_8.15 (Q0)
- new net DVY12: D_6.2 (Q0)
- new net DVY2: F_8.14 (Q1)
- new net DVY3: F_8.15 (Q0), J_8.7 (Dsl)
- new net DVY4: J_8.12 (Q3)
- new net DVY5: J_8.13 (Q2)
- new net DVY6: J_8.14 (Q1)
- new net DVY7: H_8.7 (Dsl), J_8.15 (Q0)
- new net DVY8: H_8.12 (Q3)
- new net DVY9: H_8.13 (Q2)
- new net GND: A_8.7 (Dsl), A_8.8 (GND), B_8.8 (GND), C_6.8 (GND), C_8.8 (GND), D_6.8 (GND), E_7.7 (GND), F_7.7 (GND), F_8.7 (Dsl), F_8.8 (GND), H_8.8 (GND), J_8.8 (GND)
- new net OP0: D_6.7 (Q1)
- new net OP1: D_6.10 (Q2)
- new net OP2: D_6.15 (Q3)
- new net PR82: A_8.2 (Dsr), B_8.2 (Dsr), C_8.2 (Dsr), D_6.1 (~{Mr}), F_8.2 (Dsr), H_8.1 (Mr), H_8.2 (Dsr), J_8.2 (Dsr)
- new net Z0: C_6.7 (Q1)
- new net Z1: C_6.10 (Q2)
- new net Z2: C_6.15 (Q3)
- new net ~{DVX12}: C_6.3 (~{Q0})
- new net ~{DVY12}: D_6.3 (~{Q0})
- new net ~{ENORM}: E_7.1, E_7.10, E_7.13, E_7.5
- new net ~{LATCH0}: E_7.2, F_7.13
- new net ~{LATCH1}: A_8.1 (Mr), B_8.1 (Mr), C_6.1 (~{Mr}), C_8.1 (Mr), D_6.9 (Cp), E_7.4, F_7.1, F_8.1 (Mr), J_8.1 (Mr)
- new net ~{LATCH2}: E_7.12, F_7.11
- new net ~{LATCH3}: C_6.9 (Cp), E_7.9, F_7.9
- new net ~{OP0}: D_6.6 (~{Q1})
- new net ~{OP1}: D_6.11 (~{Q2})
- new net ~{OP2}: D_6.14 (~{Q3})
- new net ~{Z1}: C_6.11 (~{Q2})
- new net ~{Z2}: C_6.14 (~{Q3})
- no-connect marks 0 -> 4
Other:
- note added: "OP CODE AND INTENSITY LATCHES"
- note added: "VECTOR DATA SHIFTERS"
