File: PCB/atari_gravitar_bw_pcb/Sheet7B.kicad_sch (KiCad schematic)
At the start: 0 parts

Commit message: Finished sheet 7B
Parts:
- added C118: 220pf, symbol Device:C
- added E_6, H_6, K_10: 74LS175, symbol atari:74LS175
- added F_5: 74LS11, symbol atari:74LS11
- added F_6: 74LS157, symbol atari:74LS157
- added H_5: 74LS20, symbol atari:74LS20
- added J_3: 74LS04, symbol atari:74LS04
- added L_10: 74LS33, symbol atari:74LS33
- added M_3: 74LS164, symbol atari:74LS164
- added M_5: 74LS32, symbol atari:74LS32
- added N_5: 74LS02, symbol atari:74LS02
- added Q10, Q5, Q6, Q8, Q9: 2N3904, Package_TO_SOT_THT:TO-92_Inline, symbol Transistor_BJT:2N3904
- added Q7: 2N3906, Package_TO_SOT_THT:TO-92_Inline, symbol Transistor_BJT:2N3906
- added R149, R150, R152, R156: 1k, symbol Device:R_US
- added R151, R154, R158: 470, symbol Device:R_US
- added R153: 68, symbol Device:R_US
- added R155: 22k, symbol Device:R_US
- added R157: 27, symbol Device:R_US
- added R56: 4.7k, symbol Device:R_US
- added R57: 2.2k, symbol Device:R_US
- added R58: 10k, symbol Device:R_US
- added R59: 1.2k, symbol Device:R_US
- added R60: 3.9k, symbol Device:R_US
- added TPBLUE1, TPGREEN1, TPRED1, TPZOUT1: tp_2_pin, symbol atari:tp_2_pin
Connections:
- new net: Q7.2 (B), R155.2, R56.2, R57.2, R58.2, R59.2, R60.1
- new net: Q5.3 (C), Q7.3 (C), Q9.2 (B), R149.1, R152.1, R153.2, R156.1
- new net: K_10.11 (~{Q2}), L_10.11
- new net: K_10.3 (~{Q0}), L_10.2
- new net: K_10.6 (~{Q1}), L_10.9
- new net: C118.2, Q5.2 (B), R150.2
- new net: F_5.12, F_6.1 (S)
- new net: E_6.7 (Q1), F_6.10 (I1c)
- new net: F_6.12 (Zd), H_6.4 (D0)
- new net: E_6.15 (Q3), F_6.13 (I1d)
- new net: E_6.2 (Q0), F_6.3 (I1a)
- new net: F_6.4 (Za), H_6.13 (D3)
- new net: E_6.10 (Q2), F_6.6 (I1b)
- new net: F_6.7 (Zb), H_6.12 (D2)
- new net: F_6.9 (Zc), H_6.5 (D1)
- new net: H_6.2 (Q0), R56.1
- new net: M_3.10 (QE), N_5.11
- new net: M_3.11 (QF), N_5.12
- new net: L_10.13, Q10.2 (B), R156.2
- new net: L_10.10, Q8.2 (B), R152.2
- new net: L_10.1, Q6.2 (B), R149.2
- new net: L_10.12, L_10.3, L_10.8, M_5.11
- new net: C118.1, M_5.13, N_5.13, R150.1
- new net: H_5.8, J_3.1
- new net: J_3.2, M_5.12
- new net: H_6.10 (Q2), R58.1
- new net: H_6.7 (Q1), R57.1
- new net: H_5.10, H_6.3 (~{Q0})
- new net: H_5.12, H_6.14 (~{Q3})
- new net: H_5.13, H_6.11 (~{Q2})
- new net: H_5.9, H_6.6 (~{Q1})
- new net: H_6.15 (Q3), R59.1
- new net +5V: E_6.16 (VCC), F_5.14 (VCC), F_6.16 (VCC), H_6.16 (VCC), J_3.14 (VCC), K_10.16 (VCC), L_10.14 (VCC), M_3.14 (VCC), Q10.3 (C), Q6.3 (C), Q8.3 (C), Q9.3 (C), R153.1, R60.2
- new net 3MHZ: M_3.8 (CLK)
- new net BLUE: Q10.1 (E), R158.2, TPBLUE1.1, TPBLUE1.2
- new net DVY0: K_10.12 (D2)
- new net DVY1: K_10.5 (D1)
- new net DVY2: K_10.4 (D0)
- new net DVY4: E_6.12 (D2)
- new net DVY5: E_6.13 (D3)
- new net DVY6: E_6.5 (D1)
- new net DVY7: E_6.4 (D0)
- new net GND: E_6.8 (GND), F_5.7 (GND), F_6.15 (E), F_6.5 (I0b), F_6.8 (GND), H_6.8 (GND), J_3.7 (GND), K_10.8 (GND), L_10.7 (GND), M_3.7 (GND), Q5.1 (E), Q7.1 (E), R151.1, R154.1, R155.1, R157.1, R158.1
- new net GREEN: Q8.1 (E), R154.2, TPGREEN1.1, TPGREEN1.2
- new net RED: Q6.1 (E), R151.2, TPRED1.1, TPRED1.2
- new net VCTR: H_6.9 (Cp), M_3.1 (A), M_3.2 (B)
- new net Z0: F_6.14 (I0d)
- new net Z1: F_6.11 (I0c)
- new net Z2: F_6.2 (I0a)
- new net Z_OUT: Q9.1 (E), R157.2, TPZOUT1.1, TPZOUT1.2
- new net ~{DISRST}: E_6.1 (~{Mr}), K_10.1 (~{Mr}), M_3.9 (C)
- new net ~{SA}: H_6.1 (~{Mr})
- new net ~{STATCLK}: E_6.9 (Cp), K_10.9 (Cp)
- new net ~{Z0}: F_5.13
- new net ~{Z1}: F_5.1
- new net ~{Z2}: F_5.2
- no-connect marks 0 -> 16
Other:
- note added: "R-G-B OUTPUT"
- note added: "Z INTENSITY AND BLANKING"
