File: PCB/atari_gravitar_bw_pcb/Sheet8A.kicad_sch (KiCad schematic)
At the start: 0 parts

Commit message: Completed sheet 8A
Parts:
- added A/B_11, C_11: MC1495L, symbol atari:MC1495L
- added A/B_9: AM6012, symbol atari:AM6012
- added A_10, D/E_1: TL082, symbol atari:TL082
- added B_10: LF13201, symbol atari:LF13201
- added C112, C127: 39pf, symbol Device:C
- added C113: 150pf, symbol Device:C
- added C122, C123, C124, C125, C70, C73, C76, C78, C86, C87, C88, C89: .1, symbol Device:C
- added C128: 100pf, symbol Device:C
- added C137: 1000pf, symbol Device:C
- added C71, C77: .01, symbol Device:C
- added C80: .047, symbol Device:C
- added C85: 10pf, symbol Device:C
- added CR4: 1N914, symbol Device:D
- added D_9: DAC_08, symbol atari:DAC_08
- added E_8: 74LS273, symbol atari:74LS273
- added K_9: 74LS04, symbol atari:74LS04
- added Q11: 2N3906, Package_TO_SOT_THT:TO-92_Inline, symbol Transistor_BJT:2N3906
- added Q12: 2N3904, Package_TO_SOT_THT:TO-92_Inline, symbol Transistor_BJT:2N3904
- added R100, R101: 7.5k, symbol Device:R_US
- added R159, R179: 10k, symbol Device:R_US
- added R160, R182: 1k, symbol Device:R_US
- added R161, R177: 15k, symbol Device:R_US
- added R162, R?: 7k 1%, symbol Device:R_US
- added R164: 560, symbol Device:R_US
- added R165, R166, R167, R168, R87, R88: 7.5K 1%, symbol Device:R_US
- added R169, R170, R176, R184: 470, symbol Device:R_US
- added R171, R172, R173, R174, R175, R185: 2.2k, symbol Device:R_US
- added R178, R183, R186, R89: 3.9k, symbol Device:R_US
- added R180, R94: 680, symbol Device:R_US
- added R181: 2.7k, symbol Device:R_US
- added R187: 2k, symbol Device:R_Potentiometer_US
- added R188: 5.6k, symbol Device:R_US
- added R189, R192: 10k, symbol Device:R_Potentiometer_US
- added R217, R90, R91: 100, symbol Device:R_US
- added R218: 68, symbol Device:R_US
- added R219: 6.8k, symbol Device:R_US
- added R74, R75, R76, R77, R78, R79, R80, R81: 100k, symbol Device:R_US
- added R95: 820, symbol Device:R_US
- added R98, R99: 500, symbol Device:R_Potentiometer_US
- added RV1: Varistor_US, symbol Device:Varistor_US
- added TPXOUT1: tp_2_pin, symbol atari:tp_2_pin
Connections:
- new net: C122.1, D/E_1.4 (V-)
- new net: A_10.2 (-), R100.2, R101.1
- new net: A_10.1, B_10.14, R101.2
- new net: A/B_9.18 (IO), A_10.6 (-), B_10.10, C137.1, C80.1, R99.1, R99.2
- new net: A_10.7, B_10.11, B_10.2, C80.2, R100.1
- new net: C_11.2, D/E_1.5 (+), R174.1, R188.2
- new net: C127.1, C128.1, C_11.14, D/E_1.6 (-), R173.1, R177.1
- new net: C127.2, C128.2, D/E_1.7, R177.2, R187.1, R187.2
- new net: C_11.12, C_11.8, R176.2
- new net: D_9.14 (VR+), R87.1, R88.1
- new net: C85.1, CR4.1 (K), D_9.4 (IO), R162.2, R165.1, R166.1, R167.1, R168.1, R?.2
- new net: C_11.4, R180.2, R181.2
- new net: C112.1, Q12.3 (C), R159.1, R160.1
- new net: C112.2, Q11.2 (B), R159.2
- new net: D_9.6 (B2), E_8.2 (Q0), R81.1
- new net: C_11.5, R175.1
- new net: C_11.6, R175.2
- new net: Q11.3 (C), R162.1, R164.2, R?.1
- new net: R166.2, R90.2
- new net: R188.1, R189.3
- new net: A/B_9.14 (VR+), R91.1, R94.2
- new net: R167.2, R91.2
- new net: C_11.13, R179.2
- new net: R165.2, R98.3
- new net: D/E_1.3 (+), R187.3, RV1.1
- new net: D_9.7 (B3), E_8.19 (Q7), R80.1
- new net: D/E_1.1, R217.2, R218.1
- new net: D/E_1.2 (-), R218.2, R219.2
- new net: B_10.15, B_10.3, R169.1, R170.2
- new net: C_11.9, R169.2
- new net: D_9.10 (B6), E_8.12 (Q4), R75.2
- new net: C113.2, Q12.2 (B), R161.2
- new net: A/B_11.10, R185.1
- new net: A/B_11.11, R185.2
- new net: R183.1, R192.3
- new net: B_10.1, K_9.12
- new net: C71.1, D_9.16 (C)
- new net: D_9.15 (VR-), R89.1
- new net: A/B_9.15 (VR-), R95.1
- new net: A/B_11.13, A/B_11.3, R186.2
- new net: A/B_11.4, A/B_11.9, R170.1
- new net: R168.2, R99.3
- new net: C_11.10, R178.1
- new net: C_11.11, R178.2
- new net: C_11.3, R183.2
- new net: D_9.8 (B4), E_8.5 (Q1), R79.1
- new net: A/B_11.5, R171.1, R172.1
- new net: A/B_11.6, R171.2, R172.2
- new net: D_9.5 (B1), E_8.16 (Q6), R78.1
- new net: C77.1, R94.1
- new net: D_9.11 (B7), E_8.6 (Q2), R76.2
- new net: D_9.12 (B8), E_8.15 (Q5), R77.2
- new net: D_9.9 (B5), E_8.9 (Q3), R74.2
- new net: A/B_11.12, A/B_11.8, R184.2
- new net +15V: A/B_11.2, A_10.8 (V+), B_10.13 (VCC), C123.1, C124.1, C87.1, C89.1, D/E_1.8 (V+), Q11.1 (E), R160.2, R173.2, R174.2, R182.2, R87.2, R88.2
- new net +5V: A/B_9.20 (VCC), C73.2, C78.2, D_9.13 (V+), E_8.20 (VCC)
- new net +6V: A/B_11.1, C_11.1
- new net -15V: A/B_11.7, A/B_9.17 (V-), A_10.4 (V-), B_10.4 (VEE), C125.1, C70.2, C71.2, C76.1, C86.1, C88.1, C_11.7, D_9.3 (V-)
- new net DVX10: A/B_9.4 (B4)
- new net DVX11: A/B_9.3 (B3)
- new net DVX3: A/B_9.11 (B11)
- new net DVX4: A/B_9.10 (B10)
- new net DVX5: A/B_9.9 (B9)
- new net DVX6: A/B_9.8 (B8)
- new net DVX7: A/B_9.7 (B7)
- new net DVX8: A/B_9.6 (B6)
- new net DVX9: A/B_9.5 (B5)
- new net DVY0: E_8.14 (D5)
- new net DVY1: E_8.7 (D2)
- new net DVY2: E_8.13 (D4)
- new net DVY3: E_8.8 (D3)
- new net DVY4: E_8.4 (D1)
- new net DVY5: E_8.18 (D7)
- new net DVY6: E_8.3 (D0)
- new net DVY7: E_8.17 (D6)
- new net GND: A/B_9.1 (B1), A/B_9.12 (B12), A/B_9.13 (GND), A/B_9.19 (~{IO}), A_10.3 (+), A_10.5 (+), B_10.5 (VR), C122.2, C123.2, C124.2, C125.2, C137.2, C70.1, C73.1, C76.2, C77.2, C78.1, C85.2, C86.2, C87.2, C88.2, C89.2, CR4.2 (A), D_9.2 (~{IO}), E_8.10 (GND), Q12.1 (E), R164.1, R176.1, R179.1, R180.1, R184.1, R186.1, R189.1, R189.2, R192.1, R192.2, R219.1, R74.1, R75.1, R76.1, R77.1, R78.2, R79.2, R80.2, R81.2, R89.2, R95.2, RV1.2
- new net INVERTX: B_10.16, K_9.13
- new net VCTR: C113.1, R161.1
- new net XCOR: A/B_11.14, R182.1
- new net X_OUT: R217.1, TPXOUT1.1, TPXOUT1.2
- new net YBIP: R98.1, R98.2
- new net YCOR: R181.1
- new net YREF: R90.1
- new net ~{CENTER}: B_10.9
- new net ~{DISRST}: E_8.1 (~{Mr})
- new net ~{DVX12}: A/B_9.2 (B2)
- new net ~{SCLAE_LD}: E_8.11 (Cp)
- new net ~{VCTR}: D_9.1 (TH)
- no-connect marks 0 -> 4
Other:
- note added: "DAC REFERENCE AND BIPOLAR CURRENT SOURCES"
- note added: "X-AXIS OUTPUT"
