File: PCB/atari_gravitar_bw_pcb/Sheet4A.kicad_sch (KiCad schematic)
At the start: 0 parts

Commit message: Completed sheet 4b
Parts:
- added B_1, C_1: 74LS244, symbol atari:74LS244
- added C_2: 6502, symbol atari:6502
- added F_2: 74LS245, symbol atari:74LS245
- added F_3: 74S04, symbol atari:74LS04
- added J_3: 74LS04, symbol atari:74LS04
- added J_4: 74LS161, symbol atari:74LS161
- added K_4: 74S10, symbol atari:74LS10
- added L_3, R_4: 74LS00, symbol atari:74LS00
- added P_3: 74LS138, symbol atari:74LS138
- added R19: 1k, symbol Device:R_US
- added R_1, R_2: grav_addr_decoder, symbol atari:grav_addr_decoder
- added TPPHI21, TPROM0, TPROM1, TPROM2, TPROM3, TPROM4, TPROM5, TPRW1, TPVMEM1: tp_2_pin, symbol atari:tp_2_pin
Connections:
- new net: B_1.17, C_2.34 (R/~{W}), TPPHI21.1, TPPHI21.2, TPRW1.1, TPRW1.2
- new net: C_1.11, C_2.16 (A7)
- new net: C_1.13, C_2.15 (A6)
- new net: C_1.15, C_2.14 (A5)
- new net: C_1.17, C_2.13 (A4)
- new net: C_1.2, C_2.9 (A0)
- new net: C_1.4, C_2.10 (A1)
- new net: C_1.6, C_2.11 (A2)
- new net: C_1.8, C_2.12 (A3)
- new net: B_1.4, C_2.17 (A8)
- new net: B_1.6, C_2.18 (A9)
- new net: C_2.2 (READY), C_2.38 (SO), C_2.6 (~{NMI}), R19.2
- new net: B_1.13, C_2.20 (A11)
- new net: B_1.15, C_2.22 (A12)
- new net: B_1.11, C_2.39 (PHI2)
- new net: C_2.4 (~{IRQ}), J_4.10 (CET), L_3.11
- new net: F_2.19 (G), R_4.3
- new net: J_4.11 (Q3), L_3.12
- new net: J_4.12 (Q2), L_3.13
- new net +5V: B_1.20 (VCC), C_1.20 (VCC), C_2.8 (VCC), F_2.20 (VCC), F_3.14 (VCC), J_4.16 (VCC), P_3.16 (VCC), R19.1, R_1.16 (VCC), R_2.16 (VCC), R_4.14 (VCC)
- new net 1.5MHZ: B_1.2, C_2.37 (PHI0)
- new net 3KHZ: J_4.2 (CP)
- new net 3MHZ: K_4.3
- new net A10: B_1.8, C_2.19 (A10)
- new net A13: C_2.23 (A13), J_3.9, R_1.12 (A2), R_2.12 (A2)
- new net A14: C_2.24 (A14), R_1.13 (A3), R_2.13 (A3)
- new net A15: C_2.25 (A15), R_1.14 (A4), R_2.14 (A4)
- new net AB0: C_1.18
- new net AB1: C_1.16
- new net AB10: B_1.12
- new net AB11: B_1.7, R_1.10 (A0), R_2.10 (A0)
- new net AB12: B_1.5, R_1.11 (A1), R_2.11 (A1)
- new net AB2: C_1.14
- new net AB3: C_1.12
- new net AB4: C_1.3
- new net AB5: C_1.5
- new net AB6: C_1.7, P_3.1 (A0)
- new net AB7: C_1.9, P_3.2 (A1)
- new net AB8: B_1.16, P_3.3 (A2)
- new net AB9: B_1.14
- new net BPHI2: B_1.9, F_3.13, K_4.5
- new net D0: C_2.33 (D0), F_2.18
- new net D1: C_2.32 (D1), F_2.17
- new net D2: C_2.31 (D2), F_2.16
- new net D3: C_2.30 (D3), F_2.15
- new net D4: C_2.29 (D4), F_2.14
- new net D5: C_2.28 (D5), F_2.13
- new net D6: C_2.27 (D6), F_2.12
- new net D7: C_2.26 (D7), F_2.11
- new net DB0: F_2.2
- new net DB1: F_2.3
- new net DB2: F_2.4
- new net DB3: F_2.5
- new net DB4: F_2.6
- new net DB5: F_2.7
- new net DB6: F_2.8
- new net DB7: F_2.9
- new net GND: B_1.1 (1G), B_1.10 (GND), B_1.19 (2G), C_1.1 (1G), C_1.10 (GND), C_1.19 (2G), C_2.1 (VSS), C_2.21 (VSS), F_2.10 (GND), F_3.7 (GND), J_4.3 (D0), J_4.4 (D1), J_4.5 (D2), J_4.6 (D3), J_4.8 (GND), P_3.8 (GND), R_1.15 (E), R_1.8 (GND), R_2.15 (E), R_2.8 (GND), R_4.7 (GND)
- new net PR23: J_4.7 (CEP), J_4.9 (~{PE}), P_3.6 (E3)
- new net ROM: R_1.2 (B1), R_4.1
- new net R~{W}B: B_1.3, F_2.1 (D/R), F_3.1
- new net VGCK: B_1.18
- new net ~{AB13}: J_3.8
- new net ~{BPHI2}: F_3.12
- new net ~{EAROMCON: P_3.11 (O4)
- new net ~{EAROMRD}: R_2.5 (B4)
- new net ~{EAROMWR: P_3.10 (O5)
- new net ~{INTACK}: J_4.1 (~{MR})
- new net ~{INTACT: P_3.12 (O3)
- new net ~{IO0}: R_2.2 (B1)
- new net ~{IO1}: R_2.3 (B2)
- new net ~{IOS}: R_2.4 (B3), R_4.2
- new net ~{IO}: P_3.4 (E1), R_2.9 (B7)
- new net ~{LATCH: P_3.15 (O0)
- new net ~{RAM}: R_2.1 (B0)
- new net ~{RESET}: C_2.40 (~{RESET})
- new net ~{ROM0}: R_1.3 (B2), TPROM0.1, TPROM0.2
- new net ~{ROM1}: R_1.4 (B3), TPROM1.1, TPROM1.2
- new net ~{ROM2}: R_1.5 (B4), TPROM2.1, TPROM2.2
- new net ~{ROM3}: R_1.6 (B5), TPROM3.1, TPROM3.2
- new net ~{ROM4}: R_1.7 (B6), TPROM4.1, TPROM4.2
- new net ~{ROM5}: R_1.9 (B7), TPROM5.1, TPROM5.2
- new net ~{R}WB: F_3.2, K_4.4
- new net ~{SINP1}: R_2.6 (B5)
- new net ~{SINP2}: R_2.7 (B6)
- new net ~{VGGO: P_3.14 (O1)
- new net ~{VGRST: P_3.13 (O2)
- new net ~{VMEM}: R_1.1 (B0), TPVMEM1.1, TPVMEM1.2
- new net ~{WDCLR}: P_3.9 (O6)
- new net ~{WRITE}: K_4.6, P_3.5 (E2)
- no-connect marks 0 -> 6
Other:
- note added: "ADDRESS DECODER"
- note added: "MICROPROCESSOR"

Commit message: Finished sheet 7B
Changed lines of the file:
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@@
     (pin "2")
   )
-  (symbol (lib_name "74LS244_1") (lib_id "atari:74LS244") (at 169.545 107.315 0) (unit 1)
+  (symbol (lib_id "atari:74LS244") (at 169.545 107.315 0) (unit 1)
     (in_bom yes) (on_board yes)
     (property "Reference" "B_1" (id 0) (at 167.005 106.045 0)

Commit message: Completed sheet 6B
Parts:
- removed R_4: 74LS00, symbol atari:74LS00
- added R_4: 74LS32, symbol atari:74LS32
Connections:
- net +5V: now also R_4.14 (VCC)
- net GND: now also R_4.7 (GND)
- net ROM: now also R_4.1
- net ~{IOS}: now also R_4.2
- net at F_2.19 (G): now also R_4.3
Changed lines of the file:
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@@
     (pin "1")
-  )
-  (symbol (lib_id "atari:74LS00") (at 146.685 221.615 0) (mirror x) (unit 1) (convert 2)
-    (in_bom yes) (on_board yes)
-    (property "Reference" "R_4" (id 0) (at 147.955 214.63 0))
-    (property "Value" "74LS00" (id 1) (at 149.86 228.6 0))
-    (property "Footprint" "" (id 2) (at 146.685 221.615 0)
-      (effects (font (size 1.27 1.27)) hide)
-    )
-    (property "Datasheet" "" (id 3) (at 146.685 221.615 0)
-      (effects (font (size 1.27 1.27)) hide)
-    )
-    (pin "1")
-    (pin "2")
-    (pin "3")
   )
   (symbol (lib_id "power:GND") (at 315.595 189.23 0) (unit 1)
@@
     )
     (pin "1")
-  )
-  (symbol (lib_id "atari:74LS00") (at 145.415 221.615 0) (unit 5)
-    (in_bom yes) (on_board yes)
-    (property "Reference" "R_4" (id 0) (at 145.415 216.535 0)
-      (effects (font (size 1.27 1.27)) (justify left))
-    )
-    (property "Value" "74LS00" (id 1) (at 146.05 226.695 0)
-      (effects (font (size 1.27 1.27)) (justify left))
-    )
-    (property "Footprint" "" (id 2) (at 145.415 221.615 0)
-      (effects (font (size 1.27 1.27)) hide)
-    )
-    (property "Datasheet" "" (id 3) (at 145.415 221.615 0)
-      (effects (font (size 1.27 1.27)) hide)
-    )
-    (pin "14")
-    (pin "7")
   )
   (symbol (lib_id "power:+5V") (at 173.99 128.905 0) (unit 1)
@@
     (pin "13")
   )
+  (symbol (lib_id "atari:74LS32") (at 146.685 221.615 0) (mirror x) (unit 1)
+    (in_bom yes) (on_board yes)
+    (property "Reference" "R_4" (id 0) (at 150.495 215.265 0))
+    (property "Value" "74LS32" (id 1) (at 149.86 228.6 0))
+    (property "Footprint" "" (id 2) (at 146.685 221.615 0)
+      (effects (font (size 1.27 1.27)) hide)
+    )
+    (property "Datasheet" "" (id 3) (at 146.685 221.615 0)
+      (effects (font (size 1.27 1.27)) hide)
+    )
+    (pin "1")
+    (pin "2")
+    (pin "3")
+  )
+  (symbol (lib_id "atari:74LS32") (at 145.415 221.615 0) (unit 5)
+    (in_bom yes) (on_board yes)
+    (property "Reference" "R_4" (id 0) (at 147.955 217.17 0)
+      (effects (font (size 1.27 1.27)) (justify left))
+    )
+    (property "Value" "74LS32" (id 1) (at 146.05 226.695 0)
+      (effects (font (size 1.27 1.27)) (justify left))
+    )
+    (property "Footprint" "" (id 2) (at 145.415 221.615 0)
+      (effects (font (size 1.27 1.27)) hide)
+    )
+    (property "Datasheet" "" (id 3) (at 145.415 221.615 0)
+      (effects (font (size 1.27 1.27)) hide)
+    )
+    (pin "14")
+    (pin "7")
+  )
   (symbol (lib_id "power:GND") (at 114.3 196.85 0) (unit 1)
