File: PCB/atari_gravitar_bw_pcb/Sheet6B.kicad_sch (KiCad schematic)
At the start: 0 parts

Commit message: Completed sheet 8A
Parts:
- added A_7, K_3: 74LS74, symbol atari:74LS74
- added B_7: 74S02, symbol atari:74LS02
- added H_7: 74LS42, symbol atari:74LS42
- added J_5: 74S260, symbol atari:74LS260
- added J_9: AVG, symbol atari:AVG
- added K_5, K_6, N_5: 74LS02, symbol atari:74LS02
- added L_4: 74LS08, symbol atari:74LS08
- added M_4: 74LS27, symbol atari:74LS27
- added N_3, R_3: 74LS157, symbol atari:74LS157
- added N_4: State_ROM, symbol atari:State_ROM
- added P_4: 74LS174, symbol atari:74LS174
- added R_4: 74LS32, symbol atari:74LS32
- added TPSACLK1: tp_2_pin, symbol atari:tp_2_pin
Connections:
- new net: A_7.13 (~{R}), R_4.8
- new net: P_4.10 (Q3), R_3.11 (I0c)
- new net: N_4.10 (Q3), P_4.11 (D3)
- new net: P_4.12 (Q4), R_3.2 (I0a)
- new net: N_4.12 (Q1), P_4.13 (D4)
- new net: N_4.11 (Q2), P_4.4 (D1)
- new net: P_4.5 (Q1), R_3.5 (I0b)
- new net: N_4.9 (Q4), P_4.6 (D2)
- new net: P_4.7 (Q2), R_3.14 (I0d)
- new net: A_7.6 (~{Q}), P_4.9 (Cp)
- new net: K_5.11, M_4.12
- new net: J_5.12, J_5.13, K_5.1, K_5.12
- new net: K_5.13, K_5.2
- new net: A_7.12 (D), A_7.2 (D), B_7.13
- new net: A_7.8 (~{Q}), H_7.12 (A3)
- new net: B_7.10, B_7.11
- new net: B_7.12, J_5.5
- new net: K_3.9 (Q), K_5.3, M_4.10
- new net: J_9.35 (ST2), L_4.6
- new net: N_3.4 (Za), N_4.1 (A6)
- new net: N_3.12 (Zd), N_4.15 (A7)
- new net: N_3.7 (Zb), N_4.2 (A5)
- new net: N_3.9 (Zc), N_4.3 (A4)
- new net: N_4.4 (A3), R_3.12 (Zd)
- new net: N_4.5 (A0), R_3.4 (Za)
- new net: N_4.6 (A1), R_3.7 (Zb)
- new net: N_4.7 (A2), R_3.9 (Zc)
- new net: K_3.12 (D), K_6.4
- new net: A_7.5 (Q), B_7.9
- new net: N_3.14 (I0d), N_5.10
- new net +5V: A_7.14 (VCC), H_7.16 (VCC), J_5.14 (VCC), J_9.37 (VDD), K_5.14 (VCC), N_3.16 (VCC), N_4.16 (VCC), P_4.16 (VCC), R_3.16 (VCC)
- new net 12MHZ: A_7.11 (C), A_7.3 (C)
- new net 3MHZ: J_5.2, K_6.6
- new net 6MHZ: J_5.3, K_3.11 (C)
- new net AVG0: J_9.36 (AVG0)
- new net AVG1: J_9.39 (AVG1)
- new net AVG10: J_9.19 (AVG10)
- new net AVG11: J_9.20 (AVG11)
- new net AVG12: J_9.21 (AVG12)
- new net AVG13: J_9.22 (AVG13)
- new net AVG2: J_9.40 (AVG2)
- new net AVG3: J_9.1 (AVG3)
- new net AVG4: J_9.2 (AVG4)
- new net AVG5: J_9.3 (AVG5)
- new net AVG6: J_9.15 (AVG6)
- new net AVG7: J_9.16 (AVG7)
- new net AVG8: J_9.17 (AVG8)
- new net AVG9: J_9.18 (AVG9)
- new net GND: A_7.7 (GND), H_7.8 (GND), J_5.7 (GND), J_9.14 (GND), K_5.7 (GND), N_3.15 (E), N_3.8 (GND), N_4.13, N_4.14, N_4.8 (GND), P_4.8 (GND), R_3.15 (E), R_3.8 (GND)
- new net GO: N_5.9
- new net HALT: P_4.3 (D0)
- new net PR23: K_3.10 (~{S}), K_3.13 (~{R})
- new net PR82: A_7.1 (~{R}), A_7.10 (~{S}), A_7.4 (~{S})
- new net SA: N_3.1 (S), R_3.1 (S)
- new net ST2: H_7.13 (A2), M_4.11
- new net VGCLK: B_7.8, J_5.1, K_6.5, TPSACLK1.1, TPSACLK1.2
- new net ~{DISRST}: P_4.1 (~{Mr})
- new net ~{VMEM}: M_4.9
- no-connect marks 0 -> 6

Commit message: Completed sheet 6B
Parts:
- added J_3: 74LS04, symbol atari:74LS04
- added R20: 10k, symbol Device:R_US
- added unit 2 of R_4
- added TPSA1: tp_2_pin, symbol atari:tp_2_pin
Connections:
- net +5V: now also R20.2
- net SA: now also R_4.10, J_3.12, R_4.5, TPSA1.1, TPSA1.2
- net ST2: now also L_4.4, N_4.10 (Q3), P_4.11 (D3)
- net at R_4.9: now also N_4.9 (Q4), P_4.6 (D2)
- net at N_4.12 (Q1), P_4.13 (D4): now also H_7.15 (A0)
- net at P_4.2 (Q0): now also N_5.8
- net at N_4.11 (Q2), P_4.4 (D1): now also H_7.14 (A1)
- net at A_7.8 (~{Q}), H_7.12 (A3): now also J_9.38 (ST3)
- net DVY6: now reaches J_9.10 (DVY6)
- net DVY7: now reaches J_9.11 (DVY7)
- net DVY8: now reaches J_9.12 (DVY8)
- net DVY9: now reaches J_9.13 (DVY9)
- net ~{STROBE0}: now reaches J_9.24 (~{STROBE0})
- net ~{STROBE0}: now also H_7.5 (4)
- net ~{OP0}: now reaches J_9.25 (~{OPX})
- net ~{OP0}: now also J_9.26 (~{OP0})
- net DVY12: now reaches J_9.27 (DVY12)
- net DVY11: now reaches J_9.28 (DVY11)
- net DVY10: now reaches J_9.29 (DVY10)
- net DVY2: now reaches J_9.30 (DVY2)
- net DVY1: now reaches J_9.31 (DVY1)
- net DVY0: now reaches J_9.32 (DVY0)
- net OP1: now reaches J_9.33 (OP1)
- net OP1: now also N_3.5 (I0b)
- net ~{STROBE1}: now reaches J_9.34 (~{STROBE1})
- net ~{STROBE1}: now also H_7.6 (5)
- net ~{STROBE2}: now reaches J_9.4 (~{STROBE2})
- net ~{STROBE2}: now also H_7.7 (6)
- net at J_9.5 (~{OP2}): now also R_4.6
- net ~{VGGO}: now reaches J_9.6 (~{VGGO})
- net DVY3: now reaches J_9.7 (DVY3)
- net DVY4: now reaches J_9.8 (DVY4)
- net DVY5: now reaches J_9.9 (DVY5)
- net at L_4.5: now also J_3.13, R20.1
- net ~{LATCH0}: now reaches H_7.1 (0)
- net ~{LATCH1}: now reaches H_7.2 (1)
- net ~{LATCH2}: now reaches H_7.3 (2)
- net ~{LATCH3}: now reaches H_7.4 (3)
- net ~{STROBE3}: now reaches H_7.9 (7)
- net AM2: now reaches R_3.10 (I1c)
- net AM3: now reaches R_3.13 (I1d)
- net AM0: now reaches R_3.3 (I1a)
- net AM1: now reaches R_3.6 (I1b)
- net AM4: now reaches N_3.10 (I1c)
- net OP0: now reaches N_3.11 (I0c)
- net AM7: now reaches N_3.13 (I1d)
- net OP2: now reaches N_3.2 (I0a)
- net AM6: now reaches N_3.3 (I1a)
- net AM5: now reaches N_3.6 (I1b)
- new net ~{OP2}: R_4.4
- no-connect marks 6 -> 7
Other:
- note added: "ADDRESS CONTROLLER"
- note added: "DECODER DISABLE"
- note added: "SIGNATURE ANALYSIS FLAG"
- note added: "STATE MACHINE"
- note added: "STATE MACHINE CLOCK"
- note added: "STATE MACHINE CLOCK LOGIC"
